Commit message: movement function

File: data/cube/boston_box_blue.urdf (robot description, URDF)
Before this commit: robot cube, 1 links, 0 joints
Links:
- link baseLink: geometry collision box size=0.025 0.025 0.025; visual mesh filename=boston_box.obj scale=0.0125 0.0125 0.0125

File: data/cube/boston_box_green.urdf (robot description, URDF)
Before this commit: robot cube, 1 links, 0 joints
Links:
- link baseLink: geometry collision box size=0.025 0.025 0.025; visual mesh filename=boston_box.obj scale=0.0125 0.0125 0.0125

File: data/cube/boston_box_red.urdf (robot description, URDF)
Before this commit: robot cube, 1 links, 0 joints
Links:
- link baseLink: geometry collision box size=0.025 0.025 0.025; visual mesh filename=boston_box.obj scale=0.0125 0.0125 0.0125
